Commit message: 完成对RSlidar的适配

File: launch/include/config/robot(lidar).urdf.xacro (robot description, xacro)
@@ -15,8 +15,8 @@
     <origin xyz="0 0 0" rpy="0 0 0" />
   </joint>
-  <link name="rslidar"> </link>
-  <joint name="rslidar_joint" type="fixed">
+  <link name="velodyne"> </link>
+  <joint name="velodyne_joint" type="fixed">
     <parent link="chassis_link" />
-    <child link="rslidar" />
+    <child link="velodyne" />
     <origin xyz="0 0 0" rpy="0 0 0" />
   </joint>
